File: New Board/Hades/Hades.kicad_pcb (KiCad board)
At the start: 2 copper layers, 10 parts, among them J1 XT60, J2 MSPM0, J3 ESP32, U1 USBLC6-2SC6, U2 USBLC6-2SC6

Commit message: changes to the board
Parts:
- removed D1: PTVS5V0Z1USK, Diode_SMD:Nexperia_DSN1608-2_1.6x0.8mm
- removed J1: XT60, Connector_AMASS:AMASS_XT60-M_1x02_P7.20mm_Vertical
- removed J2: MSPM0, Connector_USB:USB_C_Receptacle_GCT_USB4105-xx-A_16P_TopMnt_Horizontal
- removed J3: ESP32, Connector_USB:USB_C_Receptacle_GCT_USB4105-xx-A_16P_TopMnt_Horizontal
- removed R1, R2, R3, R4: 5k1, Resistor_SMD:R_0603_1608Metric_Pad0.98x0.95mm_HandSolder
- removed U1, U2: USBLC6-2SC6, Package_TO_SOT_SMD:SOT-23-6
- added H1: MountingHole_Pad, MountingHole:MountingHole_3.2mm_M3_Pad_Via, F.Cu at (79.1, 54.1)
- added H2: MountingHole_Pad, MountingHole:MountingHole_3.2mm_M3_Pad_Via, F.Cu at (79.1, 95.9)
- added H3: MountingHole_Pad, MountingHole:MountingHole_3.2mm_M3_Pad_Via, F.Cu at (170.8, 54.2)
- added H4: MountingHole_Pad, MountingHole:MountingHole_3.2mm_M3_Pad_Via, F.Cu at (170.8, 95.8)
Other:
- board outline added: 100 x 50 mm
