File: New Board/Hades/Hades.kicad_sch (KiCad schematic)
At the start: 10 parts, among them J1 XT60, J2 MSPM0, J3 ESP32, U1 USBLC6-2SC6, U2 USBLC6-2SC6

Commit message: changes to the board
Parts:
- removed D1: PTVS5V0Z1USK, Diode_SMD:Nexperia_DSN1608-2_1.6x0.8mm, symbol Diode:PTVS5V0Z1USK
- removed J1: XT60, Connector_AMASS:AMASS_XT60-M_1x02_P7.20mm_Vertical, symbol Connector:Conn_01x02_Socket
- removed J2: MSPM0, Connector_USB:USB_C_Receptacle_GCT_USB4105-xx-A_16P_TopMnt_Horizontal, symbol Connector:USB_C_Receptacle_USB2.0_16P
- removed J3: ESP32, Connector_USB:USB_C_Receptacle_GCT_USB4105-xx-A_16P_TopMnt_Horizontal, symbol Connector:USB_C_Receptacle_USB2.0_16P
- removed R1, R2, R3, R4: 5k1, Resistor_SMD:R_0603_1608Metric_Pad0.98x0.95mm_HandSolder, symbol Device:R_Small_US
- removed U1, U2: USBLC6-2SC6, Package_TO_SOT_SMD:SOT-23-6, symbol Power_Protection:USBLC6-2SC6
Connections:
- no-connect marks 4 -> 0
Other:
- added sheet HADES BRAIN (Brain.kicad_sch)
- added sheet Hades Power Distrbution Board (PDB.kicad_sch)
- note added: "HADES BRAIN"
- note added: "HADES POWER DISTRIBUTION BOARD"
- note removed: "IIIT NR"
